File: Shark50.kicad_pcb (KiCad board)
At the start: 2 copper layers, 271.5 x 81 mm, 107 parts, among them J1 USB_B_Mini, SW1 Esc, SW10 O, SW11 P, SW12 [, SW13 ], SW14 BkSpc, SW15 Tab_125, SW16 LShift_175, SW17 LCtrl_125, SW18 A, SW19 Z, SW2 Q, SW20 S, SW21 X, SW22 LAlt_125, SW23 D, SW24 C, SW25 F, SW26 V, SW27 G, SW28 B, SW29 Space_7, SW3 W, SW30 H, SW31 N, SW32 J, SW33 M, SW34 K, SW35 <, SW36 L, SW37 >, SW38 ;, SW39 /, SW4 E, SW40 RAlt_125, SW41 ', SW42 RShift_125, SW43 Enter_175, SW44 Fn, SW45 RCtr_125, SW5 R, SW6 T, SW7 Y, SW8 U, SW9 I, U1 ATmega32U4-AU, Y1 16MHz

Commit message: Finished multi layout wiring
Parts:
- added D46: 1N4148W, Diode_SMD:D_SOD-123, F.Cu at (-182.9, 57.1)
- added D47: 1N4148W, Diode_SMD:D_SOD-123, F.Cu at (-182.9, 60.5)
- added D48: 1N4148W, Diode_SMD:D_SOD-123, F.Cu at (-182.9, 63.9)
- added D49: 1N4148W, Diode_SMD:D_SOD-123, F.Cu at (-182.9, 67.2)
- added D50: 1N4148W, Diode_SMD:D_SOD-123, F.Cu at (-321.5, 69.1)
- added D51: 1N4148W, Diode_SMD:D_SOD-123, F.Cu at (-315.7, 69.1)
- added D52: 1N4148W, Diode_SMD:D_SOD-123, F.Cu at (-310.0, 69.1)
- added D53: 1N4148W, Diode_SMD:D_SOD-123, F.Cu at (-304.2, 69.1)
- added D54: 1N4148W, Diode_SMD:D_SOD-123, F.Cu at (-298.5, 69.1)
- added SW46: Space_225, acheron_MX:MX225, B.Cu at (-190.5, -31.0)
- added SW47: Space_1, acheron_MX:MX100, B.Cu at (-159.5, -31.0)
- added SW48: Space_275, acheron_MX:MX275, B.Cu at (-123.8, -31.0)
- added SW49: Space_1, acheron_MX:MX100, B.Cu at (-88.1, -31.0)
- added SW50: Space_275, acheron_MX:MX275, B.Cu at (-185.7, -31.0)
- added SW51: Space_1, acheron_MX:MX100, B.Cu at (-150.0, -31.0)
- added SW52: Space_225, acheron_MX:MX225, B.Cu at (-119.1, -31.0)
- added SW53: Space_125, acheron_MX:MX125, B.Cu at (-85.7, -31.0)
- added SW54: Space_1, acheron_MX:MX100, B.Cu at (-64.3, -31.0)
- C1: value 22pF -> 100nF
Connections:
- C1 pad 1: Net-(C1-Pad1) -> GND
- R5 pad 2: Net-(C1-Pad1) -> Net-(R5-Pad2)
- SW29 pad 1: Col6 -> Col7
- SWP1 pad 1: Net-(C1-Pad1) -> Net-(R5-Pad2)
