File: Shark50.kicad_pcb (KiCad board)
At the start: 2 copper layers, 24 parts, among them J1 USB_B_Mini, SW1 MXSwitch, SW2 MXSwitch, SW3 MXSwitch, SW4 MXSwitch, U1 ATmega32U4-AU, Y1 16MHz

Commit message: feat: added switches layout to the PCB
Parts:
- added D10: 1N4148W, Diodes_SMD:D_SOD-123, B.Cu at (101.0, 181.2)
- added D11: 1N4148W, Diodes_SMD:D_SOD-123, B.Cu at (101.0, 178.8)
- added D12: 1N4148W, Diodes_SMD:D_SOD-123, B.Cu at (29.2, 114.0)
- added D13: 1N4148W, Diodes_SMD:D_SOD-123, B.Cu at (29.2, 111.7)
- added D14: 1N4148W, Diodes_SMD:D_SOD-123, B.Cu at (24.4, 109.3)
- added D15: 1N4148W, Diodes_SMD:D_SOD-123, B.Cu at (29.2, 109.3)
- added D16: 1N4148W, Diodes_SMD:D_SOD-123, B.Cu at (24.4, 107.0)
- added D17: 1N4148W, Diodes_SMD:D_SOD-123, B.Cu at (29.2, 107.0)
- added D18: 1N4148W, Diodes_SMD:D_SOD-123, B.Cu at (105.8, 181.2)
- added D19: 1N4148W, Diodes_SMD:D_SOD-123, B.Cu at (101.0, 176.5)
- added D20: 1N4148W, Diodes_SMD:D_SOD-123, B.Cu at (105.8, 178.8)
- added D21: 1N4148W, Diodes_SMD:D_SOD-123, B.Cu at (14.9, 94.9)
- added D22: 1N4148W, Diodes_SMD:D_SOD-123, B.Cu at (19.7, 99.5)
- added D23: 1N4148W, Diodes_SMD:D_SOD-123, B.Cu at (10.2, 90.2)
- added D24: 1N4148W, Diodes_SMD:D_SOD-123, B.Cu at (19.7, 97.1)
- added D25: 1N4148W, Diodes_SMD:D_SOD-123, B.Cu at (14.9, 92.5)
- added D26: 1N4148W, Diodes_SMD:D_SOD-123, B.Cu at (10.2, 87.8)
- added D27: 1N4148W, Diodes_SMD:D_SOD-123, B.Cu at (24.4, 104.6)
- added D28: 1N4148W, Diodes_SMD:D_SOD-123, B.Cu at (8.35, 85.5)
- added D29: 1N4148W, Diodes_SMD:D_SOD-123, B.Cu at (19.7, 94.8)
- added D30: 1N4148W, Diodes_SMD:D_SOD-123, B.Cu at (19.7, 92.4)
- added D31: 1N4148W, Diodes_SMD:D_SOD-123, B.Cu at (14.9, 90.2)
- added D32: 1N4148W, Diodes_SMD:D_SOD-123, B.Cu at (14.9, 87.8)
- added D33: 1N4148W, Diodes_SMD:D_SOD-123, B.Cu at (110.5, 181.2)
- added D34: 1N4148W, Diodes_SMD:D_SOD-123, B.Cu at (110.5, 178.8)
- added D35: 1N4148W, Diodes_SMD:D_SOD-123, B.Cu at (105.8, 176.5)
- added D36: 1N4148W, Diodes_SMD:D_SOD-123, B.Cu at (115.3, 181.2)
- added D37: 1N4148W, Diodes_SMD:D_SOD-123, B.Cu at (115.3, 178.8)
- added D38: 1N4148W, Diodes_SMD:D_SOD-123, B.Cu at (29.2, 104.6)
- added D39: 1N4148W, Diodes_SMD:D_SOD-123, B.Cu at (115.3, 176.5)
- added D40: 1N4148W, Diodes_SMD:D_SOD-123, B.Cu at (5.40, 87.8)
- added D41: 1N4148W, Diodes_SMD:D_SOD-123, B.Cu at (110.5, 176.5)
- added D42: 1N4148W, Diodes_SMD:D_SOD-123, B.Cu at (5.40, 90.2)
- added D43: 1N4148W, Diodes_SMD:D_SOD-123, B.Cu at (19.7, 90.1)
- added D44: 1N4148W, Diodes_SMD:D_SOD-123, B.Cu at (19.7, 87.7)
- added D45: 1N4148W, Diodes_SMD:D_SOD-123, B.Cu at (13.1, 85.5)
- added D5: 1N4148W, Diodes_SMD:D_SOD-123, B.Cu at (14.9, 99.6)
- added D6: 1N4148W, Diodes_SMD:D_SOD-123, B.Cu at (14.9, 97.2)
- added D7: 1N4148W, Diodes_SMD:D_SOD-123, B.Cu at (10.2, 94.9)
- added D8: 1N4148W, Diodes_SMD:D_SOD-123, B.Cu at (10.2, 92.5)
- added D9: 1N4148W, Diodes_SMD:D_SOD-123, B.Cu at (96.3, 176.5)
- added R5: 330, Resistors_SMD:R_1206_HandSoldering, B.Cu at (18.8, 85.4)
- added SW10: O, acheron_MX:MX100, B.Cu at (-97.6, -88.1)
- added SW11: P, acheron_MX:MX100, B.Cu at (-78.6, -88.1)
- added SW12: [, acheron_MX:MX100, B.Cu at (-59.5, -88.1)
- added SW13: ], acheron_MX:MX100, B.Cu at (-40.5, -88.1)
- added SW14: BkSpc, acheron_MX:MX100, B.Cu at (-21.4, -88.1)
- added SW15: Tab_125, acheron_MX:MX125, B.Cu at (-266.7, -69.1)
- added SW16: LShift_175, acheron_MX:MX175, B.Cu at (-261.9, -50.0)
- added SW17: LCtrl_125, acheron_MX:MX125, B.Cu at (-266.7, -31.0)
- added SW18: A, acheron_MX:MX100, B.Cu at (-245.3, -69.1)
- added SW19: Z, acheron_MX:MX100, B.Cu at (-235.7, -50.0)
- added SW20: S, acheron_MX:MX100, B.Cu at (-226.2, -69.1)
- added SW21: X, acheron_MX:MX100, B.Cu at (-216.7, -50.0)
- added SW22: LAlt_125, acheron_MX:MX125, B.Cu at (-223.8, -31.0)
- added SW23: D, acheron_MX:MX100, B.Cu at (-207.2, -69.1)
- added SW24: C, acheron_MX:MX100, B.Cu at (-197.6, -50.0)
- added SW25: F, acheron_MX:MX100, B.Cu at (-188.1, -69.1)
- added SW26: V, acheron_MX:MX100, B.Cu at (-178.6, -50.0)
- added SW27: G, acheron_MX:MX100, B.Cu at (-169.1, -69.1)
- added SW28: B, acheron_MX:MX100, B.Cu at (-159.5, -50.0)
- added SW29: Space_7, acheron_MX:MX700, B.Cu at (-145.3, -31.0)
- added SW30: H, acheron_MX:MX100, B.Cu at (-150.0, -69.1)
- added SW31: N, acheron_MX:MX100, B.Cu at (-140.5, -50.0)
- added SW32: J, acheron_MX:MX100, B.Cu at (-131.0, -69.1)
- added SW33: M, acheron_MX:MX100, B.Cu at (-121.4, -50.0)
- added SW34: K, acheron_MX:MX100, B.Cu at (-111.9, -69.1)
- added SW35: <, acheron_MX:MX100, B.Cu at (-102.4, -50.0)
- added SW36: L, acheron_MX:MX100, B.Cu at (-92.9, -69.1)
- added SW37: >, acheron_MX:MX100, B.Cu at (-83.3, -50.0)
- added SW38: ;, acheron_MX:MX100, B.Cu at (-73.8, -69.1)
- added SW39: /, acheron_MX:MX100, B.Cu at (-64.3, -50.0)
- added SW40: RAlt_125, acheron_MX:MX125, B.Cu at (-66.7, -31.0)
- added SW41: ', acheron_MX:MX100, B.Cu at (-54.8, -69.1)
- added SW42: RShift_125, acheron_MX:MX125, B.Cu at (-42.9, -50.0)
- added SW43: Enter_175, acheron_MX:MX175, B.Cu at (-28.6, -69.1)
- added SW44: Fn, acheron_MX:MX100, B.Cu at (-21.4, -50.0)
- added SW45: RCtr_125, acheron_MX:MX125, B.Cu at (-23.8, -31.0)
- added SW5: R, acheron_MX:MX100, B.Cu at (-192.9, -88.1)
- added SW6: T, acheron_MX:MX100, B.Cu at (-173.8, -88.1)
- added SW7: Y, acheron_MX:MX100, B.Cu at (-154.8, -88.1)
- added SW8: U, acheron_MX:MX100, B.Cu at (-135.7, -88.1)
- added SW9: I, acheron_MX:MX100, B.Cu at (-116.7, -88.1)
- C2, C3, C4, C5, C6, C7, C8, J1, SWP1, U1, Y1: moved to B.Cu
- D1: value D_Small -> 1N4148W
- D2, D3, D4: value D_Small -> 1N4148W; moved to B.Cu
- R4: value 10k -> 1k; moved to B.Cu
- SW1: value MXSwitch -> Esc
- SW2: value MXSwitch -> Q
- SW3: value MXSwitch -> W
- SW4: value MXSwitch -> E
- moved SW1 334.5 mm to (-269.1, -88.1)
- moved SW2 324.8 mm to (-250.0, -88.1)
- moved SW3 317.0 mm to (-231.0, -88.1)
- moved SW4 307.9 mm to (-211.9, -88.1)
- moved C3 46.9 mm to (119.3, 57.2), turned to 180 degrees
- moved C5 46.9 mm to (119.3, 59.0), turned to 180 degrees
- moved D2 46.7 mm to (119.2, 55.1), turned to 180 degrees
- moved SWP1 42.9 mm to (117.3, 51.0), turned to 180 degrees
- moved Y1 42.2 mm to (116.9, 46.2), turned to 180 degrees
- moved C2 29.9 mm to (110.7, 49.1), turned to 180 degrees
- moved D3 28.3 mm to (109.9, 45.5), turned to 180 degrees
- moved C4 18.1 mm to (104.7, 44.5), turned to 180 degrees
- moved R4 14.0 mm to (95.0, 50.0), turned to 180 degrees
- moved C7 13.0 mm to (89.4, 49.8), turned to 180 degrees
- moved C1 4.76 mm to (58.8, 70.1)
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Connections:
- C1 pad 1: GND -> Net-(C1-Pad1)
- D3 pad 1: Row2 -> Row1
- D4 pad 1: Row2 -> Row1
- SW3 pad 1: Col1 -> Col3
- SW4 pad 1: Col2 -> Col4
- SWP1 pad 1: GND -> Net-(C1-Pad1)
- U1 pad 3: Net-(U1-Pad3) -> Net-(R3-Pad1)
Other:
- board outline added: 271.5 x 81 mm

Commit message: feat: added USB connector to the PCB
Parts:
- moved J1 267.1 mm to (-145.3, -93.5), turned to 0 degrees
Other:
- outline, holes or cut-outs redrawn

Commit message: feat: beginning of MCU routing
Parts:
- added C10: 100n, Capacitor_SMD:C_0805_2012Metric_Pad1.15x1.40mm_HandSolder, B.Cu at (-126.2, -27.7)
- added C9: 1u, Capacitor_SMD:C_0805_2012Metric_Pad1.15x1.40mm_HandSolder, B.Cu at (-125.5, -35.2)
- C1, C2, C3, C4, C5, C6, C7, C8: footprint Capacitors_SMD:C_0805_HandSoldering -> Capacitor_SMD:C_0805_2012Metric_Pad1.15x1.40mm_HandSolder
- R2, R3: moved to B.Cu
- moved C5 253.8 mm to (-114.4, -39.9)
- moved R3 251.5 mm to (-147.3, -87.6), turned to 90 degrees
- moved R2 243.6 mm to (-143.5, -87.6), turned to 90 degrees
- moved C3 239.6 mm to (-104.1, -29.2), turned to 270 degrees
- moved C8 235.6 mm to (-121.8, -39.6), turned to 0 degrees
- moved C2 234.3 mm to (-112.1, -23.1)
- moved Y1 230.9 mm to (-100.3, -31.8), turned to 270 degrees
- moved C4 223.2 mm to (-104.1, -34.3), turned to 270 degrees
- moved C7 214.9 mm to (-107.8, -35.6), turned to 270 degrees
- moved U1 207.1 mm to (-116.8, -31.8), turned to 270 degrees
- moved D4 4.11 mm to (97.8, 27.9)
Connections:
- net Net-(R2-Pad1) renamed /DP
- net Net-(R3-Pad1) renamed /DN
- R1 pad 1: RST -> Net-(R1-Pad1)
- R5 pad 2: Net-(C1-Pad1) -> Net-(R5-Pad2)
- U1 pad 42: Net-(U1-Pad42) -> +5V
- Y1 pad 1: Net-(C4-Pad2) -> Net-(Y1-Pad1)
- Y1 pad 2: Net-(C3-Pad1) -> Net-(Y1-Pad2)
Routing:
- net GND: track 0.00 -> 168.8 mm
- net +5V: track 0.00 -> 162.0 mm, vias 0 -> 6
- net /DP: track 0.00 -> 62.9 mm
- net /DN: track 0.00 -> 62.9 mm
- net Net-(C3-Pad1): track 0.00 -> 12.0 mm
- net Net-(C4-Pad2): track 0.00 -> 11.6 mm
- net Net-(J1-Pad2): track 0.00 -> 5.33 mm
- net Net-(J1-Pad3): track 0.00 -> 4.02 mm
